Commit message: Reconfigured rover center

File: component_robot_description/urdf/leo_raph.urdf (robot description, URDF)
Before this commit: robot leo_raph_unreal, 19 links, 18 joints
Joints:
- joint base_footprint_joint: origin xyz=0.0000 0.0000 -0.2697 rpy=0.000000 0.000000 0.000000 -> xyz=0.0000 0.0000 -0.0885 rpy=0.000000 0.000000 0.000000
- joint event_camera_joint: origin xyz=0.1712 -0.0072 0.2838 rpy=-0.000000 0.349066 -0.000000 -> xyz=0.1850 0.0000 0.4650 rpy=-0.000000 0.349066 -0.000000
- joint lidar_joint: origin xyz=0.1712 -0.0072 0.2838 rpy=-0.000000 0.349066 -0.000000 -> xyz=0.1850 0.0000 0.4650 rpy=-0.000000 0.349066 -0.000000
- joint navcam_central_joint: origin xyz=0.1712 -0.0072 0.2838 rpy=-0.000000 0.349066 -0.000000 -> xyz=0.1850 0.0000 0.4650 rpy=-0.000000 0.349066 -0.000000
- joint navcam_left_joint: origin xyz=0.1712 0.0928 0.2838 rpy=-0.000000 0.349066 -0.000000 -> xyz=0.1850 0.1000 0.4650 rpy=-0.000000 0.349066 -0.000000
- joint navcam_right_joint: origin xyz=0.1712 -0.1072 0.2838 rpy=-0.000000 0.349066 -0.000000 -> xyz=0.1850 -0.1000 0.4650 rpy=-0.000000 0.349066 -0.000000
- joint rear_cam_joint: origin xyz=-0.2488 -0.0072 0.1488 rpy=0.000000 0.349066 -3.141593 -> xyz=-0.2350 0.0000 0.3300 rpy=0.000000 0.349066 -3.141593
- joint spad_joint: origin xyz=0.1712 -0.0072 0.2838 rpy=-0.000000 0.349066 -0.000000 -> xyz=0.1850 0.0000 0.4650 rpy=-0.000000 0.349066 -0.000000
- joint wheel_fl_link_joint: origin xyz=0.1812 0.1827 -0.1812 rpy=0.000000 0.000000 0.000000 -> xyz=0.1950 0.1898 -0.0000 rpy=0.000000 0.000000 0.000000
- joint wheel_fr_link_joint: origin xyz=0.1812 -0.1973 -0.1812 rpy=0.000000 0.000000 0.000000 -> xyz=0.1950 -0.1902 0.0000 rpy=0.000000 0.000000 0.000000
- joint wheel_rl_link_joint: origin xyz=-0.2088 0.1827 -0.1812 rpy=0.000000 0.000000 0.000000 -> xyz=-0.1950 0.1898 0.0000 rpy=0.000000 0.000000 0.000000
- joint wheel_rr_link_joint: origin xyz=-0.2088 -0.1973 -0.1812 rpy=0.000000 0.000000 0.000000 -> xyz=-0.1950 -0.1902 0.0000 rpy=0.000000 0.000000 0.000000
